Commit message: Setting up ros2_control
- controller manager not connecting to robot simulation

File: solo12_description/urdf/solo12.ros2_control.xacro (robot description, xacro)
@@ -2,87 +2,88 @@
 <robot xmlns:xacro="http://www.ros.org/wiki/xacro">
   <xacro:macro name="solo12_ros2_control" params="use_sim">
-      <ros2_control name="Solo12HardwareInterface" type="system">
-        <hardware>
-          <!-- If "use_sim" argument is set to true launch gazebo simulation -->
-          <xacro:if value="${use_sim}">
-            <plugin>gazebo_ros2_control/GazeboSystem</plugin>
-          </xacro:if>
-          <!--
-            Otherwise launch real hardware
-          TODO:
-          - add hardware interface for the robot
-          -->
-          <xacro:unless value="${use_sim}">
-            <plugin>placeholder_namespace/PlaceHolderClass</plugin>
-          </xacro:unless>
-        </hardware>
-        <joint name="FL_HAA">
-          <command_interface name="velocity"/>
-          <state_interface name="position"/>
-          <state_interface name="velocity"/>
-        </joint>
-        <joint name="FL_HFE">
-          <command_interface name="velocity"/>
-          <state_interface name="position"/>
-          <state_interface name="velocity"/>
-        </joint>
-        <joint name="FL_KFE">
-          <command_interface name="velocity"/>
-          <state_interface name="position"/>
-          <state_interface name="velocity"/>
-        </joint>
-        <joint name="FR_HAA">
-          <command_interface name="velocity"/>
-          <state_interface name="position"/>
-          <state_interface name="velocity"/>
-        </joint>
-        <joint name="FR_HFE">
-          <command_interface name="velocity"/>
-          <state_interface name="position"/>
-          <state_interface name="velocity"/>
-        </joint>
-        <joint name="FR_KFE">
-          <command_interface name="velocity"/>
-          <state_interface name="position"/>
-          <state_interface name="velocity"/>
-        </joint>
-        <joint name="HL_HAA">
-          <command_interface name="velocity"/>
-          <state_interface name="position"/>
-          <state_interface name="velocity"/>
-        </joint>
-        <joint name="HL_HFE">
-          <command_interface name="velocity"/>
-          <state_interface name="position"/>
-          <state_interface name="velocity"/>
-        </joint>
-        <joint name="HL_KFE">
-          <command_interface name="velocity"/>
-          <state_interface name="position"/>
-          <state_interface name="velocity"/>
-        </joint>
-        <joint name="HR_HAA">
-          <command_interface name="velocity"/>
-          <state_interface name="position"/>
-          <state_interface name="velocity"/>
-        </joint>
-        <joint name="HR_HFE">
-          <command_interface name="velocity"/>
-          <state_interface name="position"/>
-          <state_interface name="velocity"/>
-        </joint>
-        <joint name="HR_KFE">
-          <command_interface name="velocity"/>
-          <state_interface name="position"/>
-          <state_interface name="velocity"/>
-        </joint>
-      </ros2_control>
-    <xacro:if value="${use_sim}">
-      <gazebo>
-        <plugin name="gazebo_ros2_control" filename="libgazebo_ros2_control.so">
-          <parameters>$(find solo12_description)/config/solo12_controllers.yaml</parameters>
-        </plugin>
-      </gazebo>
-    </xacro:if>
+    <ros2_control name="GazeboSystem" type="system">
+      <hardware>
+        <!-- If "use_sim" argument is set to true launch gazebo simulation -->
+        <!-- <xacro:if value="${use_sim}"> -->
+        <plugin>gazebo_ros2_control/GazeboSystem</plugin>
+        <!-- </xacro:if> -->
+        <!--
+          Otherwise launch real hardware
+        TODO:
+        - add hardware interface for the robot
+        -->
+        <!-- <xacro:unless value="${use_sim}">
+          <plugin>placeholder_namespace/PlaceHolderClass</plugin>
+        </xacro:unless> -->
+      </hardware>
+      <joint name="FL_HAA">
+        <command_interface name="velocity"/>
+        <state_interface name="position"/>
+        <state_interface name="velocity"/>
+      </joint>
+      <joint name="FL_HFE">
+        <command_interface name="velocity"/>
+        <state_interface name="position"/>
+        <state_interface name="velocity"/>
+      </joint>
+      <joint name="FL_KFE">
+        <command_interface name="velocity"/>
+        <state_interface name="position"/>
+        <state_interface name="velocity"/>
+      </joint>
+      <joint name="FR_HAA">
+        <command_interface name="velocity"/>
+        <state_interface name="position"/>
+        <state_interface name="velocity"/>
+      </joint>
+      <joint name="FR_HFE">
+        <command_interface name="velocity"/>
+        <state_interface name="position"/>
+        <state_interface name="velocity"/>
+      </joint>
+      <joint name="FR_KFE">
+        <command_interface name="velocity"/>
+        <state_interface name="position"/>
+        <state_interface name="velocity"/>
+      </joint>
+      <joint name="HL_HAA">
+        <command_interface name="velocity"/>
+        <state_interface name="position"/>
+        <state_interface name="velocity"/>
+      </joint>
+      <joint name="HL_HFE">
+        <command_interface name="velocity"/>
+        <state_interface name="position"/>
+        <state_interface name="velocity"/>
+      </joint>
+      <joint name="HL_KFE">
+        <command_interface name="velocity"/>
+        <state_interface name="position"/>
+        <state_interface name="velocity"/>
+      </joint>
+      <joint name="HR_HAA">
+        <command_interface name="velocity"/>
+        <state_interface name="position"/>
+        <state_interface name="velocity"/>
+      </joint>
+      <joint name="HR_HFE">
+        <command_interface name="velocity"/>
+        <state_interface name="position"/>
+        <state_interface name="velocity"/>
+      </joint>
+      <joint name="HR_KFE">
+        <command_interface name="velocity"/>
+        <state_interface name="position"/>
+        <state_interface name="velocity"/>
+      </joint>
+    </ros2_control>
+    <!-- <xacro:if value="${use_sim}"> -->
+    <gazebo>
+      <plugin filename="libgazebo_ros2_control" name="gazebo_ros2_control">
+        <parameters>$(find solo12_description)/config/solo12_controllers.yaml</parameters>
+        <controller_manager_prefix_node_name>controller_manager</controller_manager_prefix_node_name>
+      </plugin>
+    </gazebo>
+    <!-- </xacro:if> -->
   </xacro:macro>
 </robot>
